File: air-module/kicad/air-module.sch (KiCad schematic (older format))
At the start: 39 parts, among them J1 IDC12, J2 ARM_SWD, P1 USB_OTG, U1 Alphasense_OPC-N2, U2 nRF52832, U3 Plantower_PM2.5_PMS_5003, U4 TPS2064, U5 BME280, U6 TPS79133

Commit message: Air Module PCB update
Parts:
- removed C4: 100nF, 0603_handsolder:0603_HandSoldering, symbol C
- removed J2: ARM_SWD, 10pin_50mil_header:10pin_50mil_header, symbol ARM_SWD
- added J2: ARM_SWD_SMALL, Socket_Strips:Socket_Strip_Straight_2x02, symbol ARM_SWD_SMALL
- C11: footprint 0805_handsolder:0805_HandSoldering -> 0603_handsolder:0603_HandSoldering
- R11, R12, R13, R14: value 10K -> 0R
Connections:
- net +3V3: now also J2.1 (VCC)
- net GND: now also J2.3 (GND)
- net TCK: now also J2.4 (SWDCLK)
- net TMS: now also J2.2 (SWDIO)
- net RESET: no longer names the net of R1.1, U2.1 (P0.21/nRESET)
- no-connect marks 21 -> 18
Other:
- moved on the sheet: R1, R15, R16
