File: air-module/kicad/air-module.kicad_pcb (KiCad board)
At the start: 2 copper layers, 71.1 x 41.1 mm, 39 parts, among them J1 IDC12, J2 ARM_SWD, P1 USB_OTG, U1 Alphasense_OPC-N2, U2 nRF52832, U3 Plantower_PM2.5_PMS_5003, U4 TPS2064, U5 BME280, U6 TPS79133

Commit message: Air Module PCB update
Parts:
- removed C4: 100nF, 0603_handsolder:0603_HandSoldering
- C1, C10, C9, U2: moved to B.Cu
- C11: footprint 0805_handsolder:0805_HandSoldering -> 0603_handsolder:0603_HandSoldering
- J2: value ARM_SWD -> ARM_SWD_SMALL; footprint 10pin_50mil_header:10pin_50mil_header -> Socket_Strips:Socket_Strip_Straight_2x02
- R11, R12, R13, R14: value 10K -> 0R
- moved JP2 94.9 mm to (120.8, 87.5)
- moved C3 79.8 mm to (141.0, 83.0), turned to 180 degrees
- moved C7 75.1 mm to (112.4, 91.0), turned to 180 degrees
- moved C6 73.7 mm to (112.8, 97.3)
- moved J2 68.0 mm to (141.6, 105.5), turned to 270 degrees
- moved U3 67.9 mm to (111.7, 94.3)
- moved C5 66.9 mm to (146.5, 83.0)
- moved JP1 64.8 mm to (139.4, 86.3), turned to 180 degrees
- moved C1 62.6 mm to (135.8, 106.7), turned to 270 degrees
- moved U5 58.5 mm to (147.1, 97.3), turned to 270 degrees
- moved U4 50.1 mm to (133.6, 79.1), turned to 90 degrees
- moved C2 49.8 mm to (148.3, 95.4)
- moved C8 49.7 mm to (157.9, 80.5)
- moved U6 48.8 mm to (151.2, 79.8), turned to 270 degrees
- moved C11 47.0 mm to (157.2, 83.1)
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Connections:
- R1 pad 1: RESET -> Net-(R1-Pad1)
- U2 pad 1: RESET -> Net-(R1-Pad1)
Routing:
- net GND: track 0.00 -> 127.6 mm, vias 0 -> 1
- net TWI-SCL: track 0.00 -> 85.0 mm, vias 0 -> 6
- net TWI-SDA: track 0.00 -> 68.9 mm, vias 0 -> 5
- net +3V3: track 0.00 -> 58.0 mm, vias 0 -> 2
- net +5V: track 0.00 -> 53.8 mm, vias 0 -> 1
- net OC_ALPHA: track 0.00 -> 51.7 mm, vias 0 -> 1
- net MCU-RTS: track 0.00 -> 46.7 mm
- net OC_PLANT: track 0.00 -> 43.4 mm, vias 0 -> 1
- net MCU-CTS: track 0.00 -> 41.2 mm
- net EN_ALPHA: track 0.00 -> 35.8 mm, vias 0 -> 3
- net EN_PLANT: track 0.00 -> 31.4 mm, vias 0 -> 3
- net VCC_PLANT: track 0.00 -> 31.2 mm, vias 0 -> 1
- net VCC_ALPHA: track 0.00 -> 24.1 mm, vias 0 -> 2
- net MCU-TX: track 0.00 -> 16.2 mm, vias 0 -> 1
- net MCU-RX: track 0.00 -> 15.0 mm, vias 0 -> 1
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Other:
- net class Default: clearance 0.2 -> 0.1778; trace_width 0.25 -> 0.2032
- rule trace_clearance: 0.2 -> 0.1778
- board text added: "3V3"
- board text added: "CLK"
- board text added: "DAT"
- board text added: "GND"
- board text added: "SWD"

Commit message: Air Module PCB update
Parts:
- added G***: LOGO, OPENHARDWARE:OSHWLOGO0.3IN, B.Cu at (172.0, 85.0)
- moved C1 4.17 mm to (135.8, 110.9), turned to 90 degrees
Routing:
- net GND: track 127.6 -> 308.8 mm, vias 1 -> 27
- net +3V3: track 58.0 -> 158.2 mm, vias 2 -> 7
- net MCU-RX: track 15.0 -> 82.2 mm, vias 1 -> 4
- net SPI-MOSI: track 0.00 -> 63.9 mm, vias 0 -> 2
- net SPI-MISO: track 0.00 -> 53.1 mm, vias 0 -> 3
- net SPI-CS: track 0.00 -> 51.8 mm, vias 0 -> 2
- net SPI-SCLK: track 0.00 -> 48.4 mm, vias 0 -> 3
- net TCK: track 8.79 -> 54.4 mm, vias 0 -> 1
- net TMS: track 8.01 -> 46.5 mm, vias 0 -> 1
- net MCU-TX: track 16.2 -> 50.4 mm, vias 1 -> 3
- net TWI-SDA: track 68.9 -> 76.8 mm
- net VCC_ALPHA: track 24.1 -> 30.7 mm, vias 2 -> 3
- net OC_PLANT: track 43.4 -> 49.4 mm
- net OC_ALPHA: track 51.7 -> 49.5 mm
- net Net-(R7-Pad2): track 5.70 -> 7.54 mm
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- added copper zone on B.Cu, net GND
- added copper zone on F.Cu, net GND
Other:
- board text added: "Air Module"
- board text added: "Alphasense"
- board text added: "Institute IRNAS Rače"
- board text added: "Plantower"
- board text added: "SOLARCAST"

Commit message: Air Module PCB update
Parts:
- moved C1 1.97 mm to (135.9, 108.9)
- turned C10 to 0 degrees
- turned C9 to 0 degrees
- turned D1 to 90 degrees
- turned D2 to 90 degrees
- turned R1 to 270 degrees
- turned R2 to 90 degrees
- turned R3 to 90 degrees
- turned R4 to 270 degrees
- turned R5 to 270 degrees
Routing:
- net EN_PLANT: track 32.2 -> 63.2 mm, vias 3 -> 5
- net EN_ALPHA: track 37.2 -> 67.8 mm, vias 3 -> 5
- net GND: track 308.8 -> 282.3 mm, vias 27 -> 19
- net OC_PLANT: track 49.4 -> 24.3 mm
- net OC_ALPHA: track 49.5 -> 31.9 mm, vias 1 -> 4
- net MCU-CTS: track 42.9 -> 58.5 mm, vias 0 -> 2
- net SPI-MOSI: track 63.9 -> 52.6 mm, vias 2 -> 4
- net MCU-TX: track 50.4 -> 60.5 mm
- net MCU-RTS: track 46.7 -> 56.1 mm, vias 0 -> 3
- net TCK: track 54.4 -> 46.7 mm, vias 1 -> 0
- net TWI-SCL: track 85.0 -> 77.6 mm
- net TWI-SDA: track 76.8 -> 69.5 mm, vias 5 -> 6
- net MCU-RX: track 82.2 -> 75.4 mm, vias 4 -> 2
- net Net-(R1-Pad1): track 3.96 -> 10.3 mm
- net LED-RED: track 5.38 -> 11.0 mm
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Other:
- net class Default: via_dia 0.6 -> 0.8
- rule via_min_drill: 0.3 -> 0.4
- rule via_min_size: 0.4 -> 0.8
