File: geiger-module/kicad/geiger-module.kicad_pcb (KiCad board)
At the start: 2 copper layers, 65 x 130 mm, 40 parts, among them J1 ARM_SWD_SMALL, P1 USB_OTG, Q1 BC847C, Q2 BC847C, U1 iRover, U2 TPS79133, U3 nRF52832, U4 iRover, U5 BME280

Commit message: Air Module PCB update
Parts:
- U3: moved to B.Cu
- moved U3 96.9 mm to (201.4, 62.9)
- moved J1 96.5 mm to (25.2, 132.3)
- moved U1 89.6 mm to (55.1, 130.7)
- moved P1 89.1 mm to (68.9, 73.8)
- moved U4 85.7 mm to (72.4, 127.0)
Other:
- board size 65 x 130 mm -> 92 x 65 mm
