File: geiger-module/kicad/geiger-module.sch (KiCad schematic (older format))
At the start: 26 parts

Commit message: Updated Geiger Module schematic
Parts:
- added C10, C9: 100nF, 0603_handsolder:0603_HandSoldering, symbol C
- added D2, D3: 1N4148, SOD-323_standard:SOD-323, symbol D
- added D4, D5: LED, 0603_handsolder:LED_0603_HandSoldering, symbol LED
- added Q1, Q2: BC847C, sot_32_standard:SOT-23, symbol BC847C
- added R3, R4: 1K, 0603_handsolder:0603_HandSoldering, symbol R
- added R5, R6: 100R, 0603_handsolder:0603_HandSoldering, symbol R
- added R7, R8: 100K, 0603_handsolder:0603_HandSoldering, symbol R
- D1: renamed from D?; footprint (none) -> 0603_handsolder:LED_0603_HandSoldering
- gave numbers to parts that had none: 25
Connections:
- net +3V3: now also R5.1, R6.1
- net GEIGER0: now also R3.1, R4.1
- net GND: now also C10.2, C9.2, Q1.2 (E), Q2.2 (E)
- new net: C9.1, D2.1 (K), R7.1
- new net: D2.2 (A), R3.2
- new net: Q1.1 (B), R7.2
- new net: D4.2 (A), R5.2
- new net: D4.1 (K), Q1.3 (C)
- new net: C10.1, D3.1 (K), R8.1
- new net: D3.2 (A), R4.2
- new net: Q2.1 (B), R8.2
- new net: D5.2 (A), R6.2
- new net: D5.1 (K), Q2.3 (C)
Other:
- moved on the sheet: C11, C12, J1, JP1, JP2, JP3, JP4, P1, R10, R9, U5

Commit message: Geiger Module PCB and schematic update
Parts:
- removed J1: ARM_SWD, 10pin_50mil_header:10pin_50mil_header, symbol ARM_SWD
- added J1: ARM_SWD_SMALL, Socket_Strips:Socket_Strip_Straight_2x02, symbol ARM_SWD_SMALL
- P1: footprint (none) -> DCP-USBCB-SC:DCP-USBCB-SC
- U1, U4: footprint Socket_Strips:Socket_Strip_Straight_1x03 -> B3B-PH-SM4-TB_IROVER_CONNECTOR:B3B-PH-SM4-TB_IROVER_CONNECTOR
Connections:
- net +3V3: now also J1.1 (VCC)
- net GND: now also J1.3 (GND)
- net TCK: now also J1.4 (SWDCLK)
- net TMS: now also J1.2 (SWDIO)
- net RESET: no longer names the net of R1.2, U3.1 (P0.21/nRESET)
- no-connect marks 30 -> 27
Other:
- moved on the sheet: R1
Changed lines of the file:
@@
 LIBS:irover
 LIBS:bc847c
+LIBS:arm_swd_small
 LIBS:geiger-module-cache
 EELAYER 25 0
@@
 F 0 "P1" H 9765 3470 50  0000 C CNN
 F 1 "USB_OTG" H 9440 3795 50  0000 C CNN
-F 2 "" V 9390 3495 60  0000 C CNN
+F 2 "DCP-USBCB-SC:DCP-USBCB-SC" V 9390 3495 60  0001 C CNN
 F 3 "" V 9390 3495 60  0000 C CNN
 	1    9440 3595
@@
 Text GLabel 4155 6420 3    60   Input ~ 0
 TMS
-Text GLabel 2260 5045 0    60   Input ~ 0
-RESET
 NoConn ~ 2430 5145
 NoConn ~ 2430 5345
@@
 L R R1
 U 1 1 5881651E
-P 2345 4770
-F 0 "R1" V 2425 4770 50  0000 C CNN
-F 1 "10K" V 2345 4770 50  0000 C CNN
-F 2 "0603_handsolder:0603_HandSoldering" V 2275 4770 30  0001 C CNN
-F 3 "" H 2345 4770 30  0000 C CNN
-	1    2345 4770
-	1    0    0    -1
+P 2280 5045
+F 0 "R1" V 2360 5045 50  0000 C CNN
+F 1 "10K" V 2280 5045 50  0000 C CNN
+F 2 "0603_handsolder:0603_HandSoldering" V 2210 5045 30  0001 C CNN
+F 3 "" H 2280 5045 30  0000 C CNN
+	1    2280 5045
+	0    -1   -1   0
 $EndComp
 $Comp
 L +3.3V #PWR020
 U 1 1 58816524
-P 2345 4620
-F 0 "#PWR020" H 2345 4470 50  0001 C CNN
-F 1 "+3.3V" H 2345 4760 50  0000 C CNN
-F 2 "" H 2345 4620 60  0000 C CNN
-F 3 "" H 2345 4620 60  0000 C CNN
-	1    2345 4620
-	1    0    0    -1
-$EndComp
-Wire Wire Line
-	2260 5045 2430 5045
-Wire Wire Line
-	2345 5045 2345 4920
-Connection ~ 2345 5045
+P 2130 5045
+F 0 "#PWR020" H 2130 4895 50  0001 C CNN
+F 1 "+3.3V" H 2130 5185 50  0000 C CNN
+F 2 "" H 2130 5045 60  0000 C CNN
+F 3 "" H 2130 5045 60  0000 C CNN
+	1    2130 5045
+	0    -1   -1   0
+$EndComp
 $Comp
 L GND #PWR021
@@
 $EndComp
 $Comp
-L ARM_SWD J1
-U 1 1 5881D4F4
-P 6160 2015
-F 0 "J1" H 6120 2505 60  0000 C CNN
-F 1 "ARM_SWD" H 6310 1855 60  0000 C CNN
-F 2 "10pin_50mil_header:10pin_50mil_header" H 6310 1755 60  0001 C CNN
-F 3 "" H 6160 2015 60  0000 C CNN
-	1    6160 2015
-	1    0    0    -1
-$EndComp
-$Comp
 L +3.3V #PWR030
 U 1 1 5881E283
-P 5830 1655
-F 0 "#PWR030" H 5830 1505 50  0001 C CNN
-F 1 "+3.3V" H 5830 1795 50  0000 C CNN
-F 2 "" H 5830 1655 60  0000 C CNN
-F 3 "" H 5830 1655 60  0000 C CNN
-	1    5830 1655
+P 5885 1765
+F 0 "#PWR030" H 5885 1615 50  0001 C CNN
+F 1 "+3.3V" H 5885 1905 50  0000 C CNN
+F 2 "" H 5885 1765 60  0000 C CNN
+F 3 "" H 5885 1765 60  0000 C CNN
+	1    5885 1765
 	1    0    0    -1
 $EndComp
@@
 L GND #PWR031
 U 1 1 5881EE78
-P 5715 1755
-F 0 "#PWR031" H 5715 1505 50  0001 C CNN
-F 1 "GND" H 5715 1605 50  0000 C CNN
-F 2 "" H 5715 1755 60  0000 C CNN
-F 3 "" H 5715 1755 60  0000 C CNN
-	1    5715 1755
-	0    1    1    0
-$EndComp
-Wire Wire Line
-	5715 1755 5830 1755
-Wire Wire Line
-	5770 1755 5770 1855
-Wire Wire Line
-	5770 1855 5830 1855
-Connection ~ 5770 1755
-$Comp
-L GND #PWR032
-U 1 1 5881FDAB
-P 5830 2055
-F 0 "#PWR032" H 5830 1805 50  0001 C CNN
-F 1 "GND" H 5830 1905 50  0000 C CNN
-F 2 "" H 5830 2055 60  0000 C CNN
-F 3 "" H 5830 2055 60  0000 C CNN
-	1    5830 2055
-	0    1    1    0
-$EndComp
-NoConn ~ 5830 1955
-NoConn ~ 6800 1965
-NoConn ~ 6800 1855
-Text GLabel 6800 2055 2    60   Input ~ 0
-RESET
-Text GLabel 6800 1755 2    60   Input ~ 0
+P 5885 1865
+F 0 "#PWR031" H 5885 1615 50  0001 C CNN
+F 1 "GND" H 5885 1715 50  0000 C CNN
+F 2 "" H 5885 1865 60  0000 C CNN
+F 3 "" H 5885 1865 60  0000 C CNN
+	1    5885 1865
+	1    0    0    -1
+$EndComp
+Text GLabel 6860 1865 2    60   Input ~ 0
 TCK
-Text GLabel 6800 1655 2    60   Input ~ 0
+Text GLabel 6860 1765 2    60   Input ~ 0
 TMS
 $Comp
@@
 F 0 "U1" H 1835 3845 60  0000 C CNN
 F 1 "iRover" H 1935 3425 60  0000 C CNN
-F 2 "Socket_Strips:Socket_Strip_Straight_1x03" H 1995 3505 60  0001 C CNN
+F 2 "B3B-PH-SM4-TB_IROVER_CONNECTOR:B3B-PH-SM4-TB_IROVER_CONNECTOR" H 1995 3505 60  0001 C CNN
 F 3 "" H 1995 3505 60  0000 C CNN
 	1    2095 3485
@@
 F 0 "U4" H 3680 3835 60  0000 C CNN
 F 1 "iRover" H 3780 3415 60  0000 C CNN
-F 2 "Socket_Strips:Socket_Strip_Straight_1x03" H 3840 3495 60  0001 C CNN
+F 2 "B3B-PH-SM4-TB_IROVER_CONNECTOR:B3B-PH-SM4-TB_IROVER_CONNECTOR" H 3840 3495 60  0001 C CNN
 F 3 "" H 3840 3495 60  0000 C CNN
 	1    3940 3475
@@
 $EndComp
 $Comp
-L GND #PWR033
+L GND #PWR032
 U 1 1 588237F4
 P 1405 3460
-F 0 "#PWR033" H 1405 3210 50  0001 C CNN
+F 0 "#PWR032" H 1405 3210 50  0001 C CNN
 F 1 "GND" H 1405 3310 50  0000 C CNN
 F 2 "" H 1405 3460 60  0000 C CNN
@@
 $EndComp
 $Comp
-L +3.3V #PWR034
+L +3.3V #PWR033
 U 1 1 58823800
 P 1405 3160
-F 0 "#PWR034" H 1405 3010 50  0001 C CNN
+F 0 "#PWR033" H 1405 3010 50  0001 C CNN
 F 1 "+3.3V" H 1405 3300 50  0000 C CNN
 F 2 "" H 1405 3160 60  0000 C CNN
@@
 $EndComp
 $Comp
-L GND #PWR035
+L GND #PWR034
 U 1 1 588238A9
 P 3270 3475
-F 0 "#PWR035" H 3270 3225 50  0001 C CNN
+F 0 "#PWR034" H 3270 3225 50  0001 C CNN
 F 1 "GND" H 3270 3325 50  0000 C CNN
 F 2 "" H 3270 3475 60  0000 C CNN
@@
 $EndComp
 $Comp
-L +3.3V #PWR036
+L +3.3V #PWR035
 U 1 1 588238B5
 P 3270 3175
-F 0 "#PWR036" H 3270 3025 50  0001 C CNN
+F 0 "#PWR035" H 3270 3025 50  0001 C CNN
 F 1 "+3.3V" H 3270 3315 50  0000 C CNN
 F 2 "" H 3270 3175 60  0000 C CNN
@@
 $EndComp
 $Comp
-L GND #PWR037
+L GND #PWR036
 U 1 1 588239BF
 P 2295 3425
-F 0 "#PWR037" H 2295 3175 50  0001 C CNN
+F 0 "#PWR036" H 2295 3175 50  0001 C CNN
 F 1 "GND" H 2295 3275 50  0000 C CNN
 F 2 "" H 2295 3425 60  0000 C CNN
@@
 $EndComp
 $Comp
-L +3.3V #PWR038
+L +3.3V #PWR037
 U 1 1 58823A18
 P 2295 3245
-F 0 "#PWR038" H 2295 3095 50  0001 C CNN
+F 0 "#PWR037" H 2295 3095 50  0001 C CNN
 F 1 "+3.3V" H 2295 3385 50  0000 C CNN
 F 2 "" H 2295 3245 60  0000 C CNN
@@
 $EndComp
 $Comp
-L +3.3V #PWR039
+L +3.3V #PWR038
 U 1 1 58823A71
 P 4140 3235
-F 0 "#PWR039" H 4140 3085 50  0001 C CNN
+F 0 "#PWR038" H 4140 3085 50  0001 C CNN
 F 1 "+3.3V" H 4140 3375 50  0000 C CNN
 F 2 "" H 4140 3235 60  0000 C CNN
@@
 $EndComp
 $Comp
-L GND #PWR040
+L GND #PWR039
 U 1 1 58823ACA
 P 4140 3415
-F 0 "#PWR040" H 4140 3165 50  0001 C CNN
+F 0 "#PWR039" H 4140 3165 50  0001 C CNN
 F 1 "GND" H 4140 3265 50  0000 C CNN
 F 2 "" H 4140 3415 60  0000 C CNN
@@
 $EndComp
 $Comp
-L GND #PWR041
+L GND #PWR040
 U 1 1 5880F4B5
 P 6455 3570
-F 0 "#PWR041" H 6455 3320 50  0001 C CNN
+F 0 "#PWR040" H 6455 3320 50  0001 C CNN
 F 1 "GND" H 6455 3420 50  0000 C CNN
 F 2 "" H 6455 3570 60  0000 C CNN
@@
 $EndComp
 $Comp
-L +3.3V #PWR042
+L +3.3V #PWR041
 U 1 1 58811A34
 P 6415 2840
-F 0 "#PWR042" H 6415 2690 50  0001 C CNN
+F 0 "#PWR041" H 6415 2690 50  0001 C CNN
 F 1 "+3.3V" H 6415 2980 50  0000 C CNN
 F 2 "" H 6415 2840 60  0000 C CNN
@@
 $EndComp
 $Comp
-L GND #PWR043
+L GND #PWR042
 U 1 1 5881957B
 P 7115 3395
-F 0 "#PWR043" H 7115 3145 50  0001 C CNN
+F 0 "#PWR042" H 7115 3145 50  0001 C CNN
 F 1 "GND" H 7115 3245 50  0000 C CNN
 F 2 "" H 7115 3395 60  0000 C CNN
@@
 $EndComp
 $Comp
-L GND #PWR044
+L GND #PWR043
 U 1 1 5881D6EE
 P 6525 4765
-F 0 "#PWR044" H 6525 4515 50  0001 C CNN
+F 0 "#PWR043" H 6525 4515 50  0001 C CNN
 F 1 "GND" H 6525 4615 50  0000 C CNN
 F 2 "" H 6525 4765 60  0000 C CNN
@@
 $EndComp
 $Comp
-L +3.3V #PWR045
+L +3.3V #PWR044
 U 1 1 5881D703
 P 6485 4035
-F 0 "#PWR045" H 6485 3885 50  0001 C CNN
+F 0 "#PWR044" H 6485 3885 50  0001 C CNN
 F 1 "+3.3V" H 6485 4175 50  0000 C CNN
 F 2 "" H 6485 4035 60  0000 C CNN
@@
 $EndComp
 $Comp
-L GND #PWR046
+L GND #PWR045
 U 1 1 5881D715
 P 7185 4590
-F 0 "#PWR046" H 7185 4340 50  0001 C CNN
+F 0 "#PWR045" H 7185 4340 50  0001 C CNN
 F 1 "GND" H 7185 4440 50  0000 C CNN
 F 2 "" H 7185 4590 60  0000 C CNN
@@
 	7185 4190 7185 4035
 $Comp
-L +3.3V #PWR047
+L +3.3V #PWR046
 U 1 1 58822243
 P 8020 5375
-F 0 "#PWR047" H 8020 5225 50  0001 C CNN
+F 0 "#PWR046" H 8020 5225 50  0001 C CNN
 F 1 "+3.3V" H 8020 5515 50  0000 C CNN
 F 2 "" H 8020 5375 60  0000 C CNN
@@
 $EndComp
 $Comp
-L GND #PWR048
+L GND #PWR047
 U 1 1 588222C6
 P 8015 5800
-F 0 "#PWR048" H 8015 5550 50  0001 C CNN
+F 0 "#PWR047" H 8015 5550 50  0001 C CNN
 F 1 "GND" H 8015 5650 50  0000 C CNN
 F 2 "" H 8015 5800 60  0000 C CNN
@@
 $EndComp
 $Comp
-L PWR_FLAG #FLG049
+L PWR_FLAG #FLG048
 U 1 1 588238CF
 P 8020 5375
-F 0 "#FLG049" H 8020 5470 50  0001 C CNN
+F 0 "#FLG048" H 8020 5470 50  0001 C CNN
 F 1 "PWR_FLAG" H 8020 5555 50  0000 C CNN
 F 2 "" H 8020 5375 60  0000 C CNN
@@
 $EndComp
 $Comp
-L PWR_FLAG #FLG050
+L PWR_FLAG #FLG049
 U 1 1 58823933
 P 8015 5800
-F 0 "#FLG050" H 8015 5895 50  0001 C CNN
+F 0 "#FLG049" H 8015 5895 50  0001 C CNN
 F 1 "PWR_FLAG" H 8015 5980 50  0000 C CNN
 F 2 "" H 8015 5800 60  0000 C CNN
@@
 	0    1    1    0
 $EndComp
+$Comp
+L ARM_SWD_SMALL J1
+U 1 1 58889618
+P 6210 2115
+F 0 "J1" H 6160 2590 60  0000 C CNN
+F 1 "ARM_SWD_SMALL" H 6385 2240 60  0000 C CNN
+F 2 "Socket_Strips:Socket_Strip_Straight_2x02" H 6385 2115 60  0001 C CNN
+F 3 "" H 6210 2115 60  0000 C CNN
+	1    6210 2115
+	1    0    0    -1
+$EndComp
 $EndSCHEMATC

Commit message: Air Geiger Modules PCB update
Connections:
- net GEIGER0: no longer R4.1
- net GEIGER1: now also R4.1

Commit message: Fixes #2
Parts:
- C3, C8: footprint 0603_handsolder:0603_HandSoldering -> 0805_handsolder:0805_HandSoldering
Changed lines of the file:
@@
 F 0 "C3" H 2035 1865 50  0000 L CNN
 F 1 "10uF" H 2035 1665 50  0000 L CNN
-F 2 "0603_handsolder:0603_HandSoldering" H 2048 1615 30  0001 C CNN
+F 2 "0805_handsolder:0805_HandSoldering" H 2048 1615 30  0001 C CNN
 F 3 "" H 2010 1765 60  0000 C CNN
 	1    2010 1765
@@
 F 0 "C8" H 4375 1905 50  0000 L CNN
 F 1 "10uF" H 4375 1705 50  0000 L CNN
-F 2 "0603_handsolder:0603_HandSoldering" H 4388 1655 30  0001 C CNN
+F 2 "0805_handsolder:0805_HandSoldering" H 4388 1655 30  0001 C CNN
 F 3 "" H 4350 1805 60  0000 C CNN
 	1    4350 1805
