File: communications-module/kicad/UART.sch (KiCad schematic (older format))
At the start: 21 parts, among them U11 FONA_3G, U12 TPS2064, U13 RockBLOCK, U14 SN74LV4052A, U15 TPS2064, U16 FGPMMOPA6H, U17 uFL_conn, U18 SN74LV4052A, U19 Gateway Module LORA, U20 TPS2064

Commit message: Communications Module PCB update
Other:
- note added: "UARTS !!"
Changed lines of the file:
@@
 encoding utf-8
 Sheet 4 4
-Title ""
-Date ""
-Rev ""
-Comp ""
+Title "Solarcast Communications Module"
+Date "2017-02-09"
+Rev "1.0"
+Comp "Institute IRNAS Rače"
 Comment1 ""
 Comment2 ""
@@
 	7280 2850 7280 2770
 Connection ~ 7280 2770
+Text Notes 2150 940  0    118  ~ 0
+UARTS !!
 $EndSCHEMATC

Commit message: Communications Module gerbers update
Other:
- note removed: "UARTS !!"
Changed lines of the file:
@@
 	7280 2850 7280 2770
 Connection ~ 7280 2770
-Text Notes 2150 940  0    118  ~ 0
-UARTS !!
 $EndSCHEMATC

Commit message: Communications Module schematic update
Parts:
- U12, U15, U20: value TPS2064 -> TPS2066
Connections:
- net ENABLE-FONA is gone; now on net ENABLE-FONA_ROCK: U12.3 (EN1*), U20.3 (EN1*)
- net ENABLE-ROCK is gone; now on net ENABLE-FONA_ROCK: R9.2, U15.3 (EN1*)
- net FONA_VBAT: now also U20.6 (OUT2)
- net GPS_RX: now also U18.4 (2Y3); no longer U18.1 (2Y0)
- net GPS_TX: now also U18.11 (1Y3); no longer U18.12 (1Y0)
- net LORA_CTS: now also U14.12 (1Y0); no longer U14.11 (1Y3)
- net LORA_RTS: now also U14.1 (2Y0); no longer U14.4 (2Y3)
- net LORA_RX: now also U18.1 (2Y0); no longer U18.4 (2Y3)
- net LORA_TX: now also U18.12 (1Y0); no longer U18.11 (1Y3)
- net ENABLE-FONA_ROCK: now reaches U20.4 (EN2*)
- net FONA_CTS renamed FONA_ROCK_CTS
- net FONA_ROCK_CTS: now also U13.5 (CTS)
- net FONA_RTS renamed FONA_ROCK_RTS
- net FONA_ROCK_RTS: now also U13.1 (RTS)
- net FONA_RX renamed FONA_ROCK_RX
- net FONA_ROCK_RX: now also U13.2 (RXD)
- net FONA_TX renamed FONA_ROCK_TX
- net FONA_ROCK_TX: now also U13.3 (TXD)
- net ROCK_CTS renamed AIR_CTS
- net AIR_CTS: no longer U13.5 (CTS)
- net ROCK_RTS renamed AIR_RTS
- net AIR_RTS: no longer U13.1 (RTS)
- net ROCK_RX renamed AIR_RX
- net AIR_RX: no longer U13.2 (RXD)
- net ROCK_TX renamed AIR_TX
- net AIR_TX: no longer U13.3 (TXD)
- no-connect marks 54 -> 52
Other:
- moved on the sheet: JP20, JP21, U15
