File: communications-module/kicad/communications-module.sch (KiCad schematic (older format))
At the start: 7 parts, among them U1 nRF52832, U2 CMSIS_DAP_Programmer

Commit message: Communications Module PCB update
Connections:
- net ENABLE-3V3 is gone; now on net ENABLE-BACKUP: U1.24 (NFC1/P0.09)
- net ENABLE-RESERV: now also U1.11 (P0.31/AIN7)
- no-connect marks 5 -> 4

Commit message: Communications Module schematic update
Parts:
- added P1: DEBUG UART, Socket_Strips:Socket_Strip_Straight_1x05_Pitch2.54mm, symbol CONN_01X05
Connections:
- net GND: now also P1.1 (P1)
- net UART_CTS: now also P1.2 (P2)
- net UART_RTS: now also P1.3 (P3)
- net UART_RX: now also P1.5 (P5)
- net UART_TX: now also P1.4 (P4)
- net ENABLE_ROCK: no longer names the net of U1.34 (P0.19)
- no-connect marks 4 -> 5
Other:
- moved on the sheet: U2
