File: communications-module/kicad/power_supply.sch (KiCad schematic (older format))
At the start: 19 parts, among them J1 IDC12, P2 USB_A, P3 USB_A, P4 USB_A, P5 BACKUP, U3 TPS2064, U4 PWR_CONN, U5 TPS2064

Commit message: Communications Module schematic update
Parts:
- U3, U5: value TPS2064 -> TPS2066
Connections:
- net UART_CTS: no longer J1.11
- net UART_RTS: no longer J1.12
- net UART_RX: no longer J1.10
- net UART_TX: no longer J1.9
- new net AIR_CTS: J1.11
- new net AIR_RTS: J1.12
- new net AIR_RX: J1.10
- new net AIR_TX: J1.9
Changed lines of the file:
@@
 TWI_SDA
 $Comp
-L GND #PWR29
+L GND #PWR041
 U 1 1 589845A1
 P 4785 2270
-F 0 "#PWR29" H 4785 2020 50  0001 C CNN
+F 0 "#PWR041" H 4785 2020 50  0001 C CNN
 F 1 "GND" H 4785 2120 50  0000 C CNN
 F 2 "" H 4785 2270 60  0000 C CNN
@@
 $EndComp
 $Comp
-L GND #PWR30
+L GND #PWR042
 U 1 1 589845A7
 P 5935 2270
-F 0 "#PWR30" H 5935 2020 50  0001 C CNN
+F 0 "#PWR042" H 5935 2020 50  0001 C CNN
 F 1 "GND" H 5935 2120 50  0000 C CNN
 F 2 "" H 5935 2270 60  0000 C CNN
@@
 TWI_SCL
 $Comp
-L GND #PWR32
+L GND #PWR043
 U 1 1 589859EA
 P 6250 5030
-F 0 "#PWR32" H 6250 4780 50  0001 C CNN
+F 0 "#PWR043" H 6250 4780 50  0001 C CNN
 F 1 "GND" H 6250 4880 50  0000 C CNN
 F 2 "" H 6250 5030 60  0000 C CNN
@@
 $EndComp
 $Comp
-L GND #PWR40
+L GND #PWR044
 U 1 1 589859F7
 P 8315 5430
-F 0 "#PWR40" H 8315 5180 50  0001 C CNN
+F 0 "#PWR044" H 8315 5180 50  0001 C CNN
 F 1 "GND" H 8315 5280 50  0000 C CNN
 F 2 "" H 8315 5430 60  0000 C CNN
@@
 TWI_SCL
 $Comp
-L GND #PWR41
+L GND #PWR045
 U 1 1 58985A1D
 P 8360 5030
-F 0 "#PWR41" H 8360 4780 50  0001 C CNN
+F 0 "#PWR045" H 8360 4780 50  0001 C CNN
 F 1 "GND" H 8360 4880 50  0000 C CNN
 F 2 "" H 8360 5030 60  0000 C CNN
@@
 $EndComp
 $Comp
-L GND #PWR25
+L GND #PWR046
 U 1 1 58985A2A
 P 4060 5560
-F 0 "#PWR25" H 4060 5310 50  0001 C CNN
+F 0 "#PWR046" H 4060 5310 50  0001 C CNN
 F 1 "GND" H 4060 5410 50  0000 C CNN
 F 2 "" H 4060 5560 60  0000 C CNN
@@
 GEIGER0
 $Comp
-L GND #PWR26
+L GND #PWR047
 U 1 1 58985A50
 P 4105 5160
-F 0 "#PWR26" H 4105 4910 50  0001 C CNN
+F 0 "#PWR047" H 4105 4910 50  0001 C CNN
 F 1 "GND" H 4105 5010 50  0000 C CNN
 F 2 "" H 4105 5160 60  0000 C CNN
@@
 $EndComp
 $Comp
-L GND #PWR34
+L GND #PWR048
 U 1 1 58985A5D
 P 6690 3760
-F 0 "#PWR34" H 6690 3510 50  0001 C CNN
+F 0 "#PWR048" H 6690 3510 50  0001 C CNN
 F 1 "GND" H 6690 3610 50  0000 C CNN
 F 2 "" H 6690 3760 60  0000 C CNN
@@
 	7615 4025 7740 4025
 $Comp
-L GND #PWR22
+L GND #PWR049
 U 1 1 58985A8F
 P 3065 3985
-F 0 "#PWR22" H 3065 3735 50  0001 C CNN
+F 0 "#PWR049" H 3065 3735 50  0001 C CNN
 F 1 "GND" H 3065 3835 50  0000 C CNN
 F 2 "" H 3065 3985 60  0000 C CNN
@@
 RESERV_5V
 $Comp
-L GND #PWR31
+L GND #PWR050
 U 1 1 58985AAE
 P 6205 5430
-F 0 "#PWR31" H 6205 5180 50  0001 C CNN
+F 0 "#PWR050" H 6205 5180 50  0001 C CNN
 F 1 "GND" H 6205 5280 50  0000 C CNN
 F 2 "" H 6205 5430 60  0000 C CNN
@@
 $EndComp
 $Comp
-L +5V #PWR23
+L +5V #PWR051
 U 1 1 58985ABE
 P 3925 3490
-F 0 "#PWR23" H 3925 3340 50  0001 C CNN
+F 0 "#PWR051" H 3925 3340 50  0001 C CNN
 F 1 "+5V" H 3925 3630 50  0000 C CNN
 F 2 "" H 3925 3490 60  0000 C CNN
@@
 $EndComp
 $Comp
-L +5V #PWR35
+L +5V #PWR052
 U 1 1 58985AD9
 P 7525 3230
-F 0 "#PWR35" H 7525 3080 50  0001 C CNN
+F 0 "#PWR052" H 7525 3080 50  0001 C CNN
 F 1 "+5V" H 7525 3370 50  0000 C CNN
 F 2 "" H 7525 3230 60  0000 C CNN
@@
 $EndComp
 $Comp
-L +5V #PWR36
+L +5V #PWR053
 U 1 1 58985AE6
 P 7525 3415
-F 0 "#PWR36" H 7525 3265 50  0001 C CNN
+F 0 "#PWR053" H 7525 3265 50  0001 C CNN
 F 1 "+5V" H 7525 3555 50  0000 C CNN
 F 2 "" H 7525 3415 60  0000 C CNN
@@
 5V
 $Comp
-L +5V #PWR38
+L +5V #PWR054
 U 1 1 58988CC2
 P 8200 1550
-F 0 "#PWR38" H 8200 1400 50  0001 C CNN
+F 0 "#PWR054" H 8200 1400 50  0001 C CNN
 F 1 "+5V" H 8200 1690 50  0000 C CNN
 F 2 "" H 8200 1550 60  0000 C CNN
@@
 $EndComp
 $Comp
-L +3.3V #PWR39
+L +3.3V #PWR055
 U 1 1 58989B65
 P 8215 1775
-F 0 "#PWR39" H 8215 1625 50  0001 C CNN
+F 0 "#PWR055" H 8215 1625 50  0001 C CNN
 F 1 "+3.3V" H 8215 1915 50  0000 C CNN
 F 2 "" H 8215 1775 60  0000 C CNN
@@
 TWI_SCL
 $Comp
-L +5V #PWR28
+L +5V #PWR056
 U 1 1 589845B4
 P 4265 1815
-F 0 "#PWR28" H 4265 1665 50  0001 C CNN
+F 0 "#PWR056" H 4265 1665 50  0001 C CNN
 F 1 "+5V" H 4265 1955 50  0000 C CNN
 F 2 "" H 4265 1815 60  0000 C CNN
@@
 $EndComp
 $Comp
-L +3.3V #PWR27
+L +3.3V #PWR057
 U 1 1 589845AE
 P 4110 1975
-F 0 "#PWR27" H 4110 1825 50  0001 C CNN
+F 0 "#PWR057" H 4110 1825 50  0001 C CNN
 F 1 "+3.3V" H 4110 2115 50  0000 C CNN
 F 2 "" H 4110 1975 60  0000 C CNN
@@
 BACKUP_5V
 $Comp
-L GND #PWR42
+L GND #PWR058
 U 1 1 589977EF
 P 10130 4435
-F 0 "#PWR42" H 10130 4185 50  0001 C CNN
+F 0 "#PWR058" H 10130 4185 50  0001 C CNN
 F 1 "GND" H 10130 4285 50  0000 C CNN
 F 2 "" H 10130 4435 60  0000 C CNN
@@
 AIR_5V
 $Comp
-L GND #PWR37
+L GND #PWR059
 U 1 1 58A00F9B
 P 8195 1320
-F 0 "#PWR37" H 8195 1070 50  0001 C CNN
+F 0 "#PWR059" H 8195 1070 50  0001 C CNN
 F 1 "GND" H 8195 1170 50  0000 C CNN
 F 2 "" H 8195 1320 60  0000 C CNN
@@
 $EndComp
 $Comp
-L +3.3V #PWR19
+L +3.3V #PWR060
 U 1 1 58999FE9
 P 1585 2625
-F 0 "#PWR19" H 1585 2475 50  0001 C CNN
+F 0 "#PWR060" H 1585 2475 50  0001 C CNN
 F 1 "+3.3V" H 1585 2765 50  0000 C CNN
 F 2 "" H 1585 2625 60  0000 C CNN
@@
 SPI_SCLK
 $Comp
-L GND #PWR20
+L GND #PWR061
 U 1 1 58A15D45
 P 2020 5185
-F 0 "#PWR20" H 2020 4935 50  0001 C CNN
+F 0 "#PWR061" H 2020 4935 50  0001 C CNN
 F 1 "GND" H 2020 5035 50  0000 C CNN
 F 2 "" H 2020 5185 60  0000 C CNN
@@
 	1540 5745 1345 5745
 Text GLabel 1345 5645 0    60   Input ~ 0
-UART_TX
+AIR_TX
 Text GLabel 1945 5645 2    60   Input ~ 0
-UART_RX
+AIR_RX
 Text GLabel 1345 5745 0    60   Input ~ 0
-UART_CTS
+AIR_CTS
 Text GLabel 1945 5745 2    60   Input ~ 0
-UART_RTS
+AIR_RTS
 Wire Wire Line
 	1790 5345 1945 5345
@@
 ENABLE-AIR
 $Comp
-L +5V #PWR21
+L +5V #PWR062
 U 1 1 58985A95
 P 2880 3985
-F 0 "#PWR21" H 2880 3835 50  0001 C CNN
+F 0 "#PWR062" H 2880 3835 50  0001 C CNN
 F 1 "+5V" H 2880 4125 50  0000 C CNN
 F 2 "" H 2880 3985 60  0000 C CNN
@@
 $EndComp
 $Comp
-L +5V #PWR24
+L +5V #PWR063
 U 1 1 58985ACB
 P 3925 3675
-F 0 "#PWR24" H 3925 3525 50  0001 C CNN
+F 0 "#PWR063" H 3925 3525 50  0001 C CNN
 F 1 "+5V" H 3925 3815 50  0000 C CNN
 F 2 "" H 3925 3675 60  0000 C CNN
@@
 BACKUP_5V
 $Comp
-L +5V #PWR33
+L +5V #PWR064
 U 1 1 58985A63
 P 6505 3760
-F 0 "#PWR33" H 6505 3610 50  0001 C CNN
+F 0 "#PWR064" H 6505 3610 50  0001 C CNN
 F 1 "+5V" H 6505 3900 50  0000 C CNN
 F 2 "" H 6505 3760 60  0000 C CNN
@@
 P 7140 3885
 F 0 "U5" H 6990 4135 60  0000 C CNN
-F 1 "TPS2064" H 7140 3660 60  0000 C CNN
+F 1 "TPS2066" H 7140 3660 60  0000 C CNN
 F 2 "TPS2064:TPS2064" H 7140 3585 60  0001 C CNN
 F 3 "" H 7040 3660 60  0000 C CNN
@@
 P 3515 4110
 F 0 "U3" H 3365 4360 60  0000 C CNN
-F 1 "TPS2064" H 3515 3885 60  0000 C CNN
+F 1 "TPS2066" H 3515 3885 60  0000 C CNN
 F 2 "TPS2064:TPS2064" H 3515 3810 60  0001 C CNN
 F 3 "" H 3415 3885 60  0000 C CNN
@@
 RESERV_5V
 $Comp
-L PWR_FLAG #FLG22
+L PWR_FLAG #FLG065
 U 1 1 589AC172
 P 1335 7385
-F 0 "#FLG22" H 1335 7480 50  0001 C CNN
+F 0 "#FLG065" H 1335 7480 50  0001 C CNN
 F 1 "PWR_FLAG" H 1335 7565 50  0000 C CNN
 F 2 "" H 1335 7385 60  0000 C CNN
@@
 $EndComp
 $Comp
-L PWR_FLAG #FLG23
+L PWR_FLAG #FLG066
 U 1 1 589AC39B
 P 2200 7390
-F 0 "#FLG23" H 2200 7485 50  0001 C CNN
+F 0 "#FLG066" H 2200 7485 50  0001 C CNN
 F 1 "PWR_FLAG" H 2200 7570 50  0000 C CNN
 F 2 "" H 2200 7390 60  0000 C CNN
@@
 $EndComp
 $Comp
-L PWR_FLAG #FLG24
+L PWR_FLAG #FLG067
 U 1 1 589AC824
 P 3220 7405
-F 0 "#FLG24" H 3220 7500 50  0001 C CNN
+F 0 "#FLG067" H 3220 7500 50  0001 C CNN
 F 1 "PWR_FLAG" H 3220 7585 50  0000 C CNN
 F 2 "" H 3220 7405 60  0000 C CNN
